Commit message: urdf建模优化base_link

File: src/simulation_learning/models/urdf/mbot_with_laser_camera_floor_link.urdf (robot description, URDF)
Before this commit: robot mbot, 7 links, 6 joints
Links:
- added link floor_link; visual cylinder length=0.000001 radius=0.20
Joints:
- added joint base_joint: type continuous, parent floor_link, child base_link, origin xyz=0 0 0.11 rpy=0 0 0, axis 0 1 0
