Commit message: code of xacro

File: src/simulation_learning/models/xacro/mbot_base.xacro (robot description, xacro)
@@ -1,5 +1,5 @@
 <?xml version="1.0"?>
 <robot name="mbot" xmlns:xacro="http://www.ros.org/wiki/xacro">
-    <!-- PROPERTY LIST -->
+    <!-- 属性列表 -->
     <xacro:property name="M_PI" value="3.1415926"/>
     <xacro:property name="base_radius" value="0.20"/>
@@ -9,5 +9,6 @@
     <xacro:property name="wheel_joint_y" value="0.19"/>
     <xacro:property name="wheel_joint_z" value="0.05"/>
-    <xacro:property name="caster_radius" value="0.015"/> <!-- wheel_radius - ( base_length/2 - wheel_joint_z) -->
+    <!-- wheel_radius - ( base_length/2 - wheel_joint_z) -->
+    <xacro:property name="caster_radius" value="0.015"/>
     <xacro:property name="caster_joint_x" value="0.18"/>
     <!-- Defining the colors used in this robot -->
