Commit message: 使用 Xacro 优化 URDF 模型

File: src/simulation_learning/models/xacro/mbot.xacro (robot description, xacro)
@@ -2,4 +2,4 @@
 <robot name="arm" xmlns:xacro="http://www.ros.org/wiki/xacro">
     <xacro:include filename="$(find simulation_learning)/urdf/xacro/mbot_base.xacro" />
-    <mbot_base/>
+    <mbot_base />
 </robot>

File: src/simulation_learning/models/xacro/mbot_base.xacro (robot description, xacro)
@@ -1,93 +1,6 @@
 <?xml version="1.0"?>
-<robot name="mbot" xmlns:xacro="http://www.ros.org/wiki/xacro">
-    <!-- 属性列表 -->
-    <xacro:property name="M_PI" value="3.1415926"/>
-    <xacro:property name="base_radius" value="0.20"/>
-    <xacro:property name="base_length" value="0.16"/>
-    <xacro:property name="wheel_radius" value="0.06"/>
-    <xacro:property name="wheel_length" value="0.025"/>
-    <xacro:property name="wheel_joint_y" value="0.19"/>
-    <xacro:property name="wheel_joint_z" value="0.05"/>
-    <!-- wheel_radius - ( base_length/2 - wheel_joint_z) -->
-    <xacro:property name="caster_radius" value="0.015"/>
-    <xacro:property name="caster_joint_x" value="0.18"/>
-    <!-- 颜色列表 -->
-    <material name="yellow">
-        <color rgba="1 0.4 0 1"/>
-    </material>
-    <material name="black">
-        <color rgba="0 0 0 0.95"/>
-    </material>
-    <material name="gray">
-        <color rgba="0.75 0.75 0.75 1"/>
-    </material>
-    <!-- 轮子宏定义 -->
-    <xacro:macro name="wheel" params="prefix reflect">
-        <joint name="${prefix}_wheel_joint" type="continuous">
-            <origin xyz="0 ${reflect*wheel_joint_y} ${-wheel_joint_z}" rpy="0 0 0"/>
-            <parent link="base_link"/>
-            <child link="${prefix}_wheel_link"/>
-            <axis xyz="0 1 0"/>
-        </joint>
-        <link name="${prefix}_wheel_link">
-            <visual>
-                <origin xyz="0 0 0" rpy="${M_PI/2} 0 0" />
-                <geometry>
-                    <cylinder radius="${wheel_radius}" length = "${wheel_length}"/>
-                </geometry>
-                <material name="gray" />
-            </visual>
-        </link>
-    </xacro:macro>
-    <!-- 脚轮宏定义 -->
-    <xacro:macro name="caster" params="prefix reflect">
-        <joint name="${prefix}_caster_joint" type="continuous">
-            <origin xyz="${reflect*caster_joint_x} 0 ${-(base_length/2 + caster_radius)}" rpy="0 0 0"/>
-            <parent link="base_link"/>
-            <child link="${prefix}_caster_link"/>
-            <axis xyz="0 1 0"/>
-        </joint>
-        <link name="${prefix}_caster_link">
-            <visual>
-                <origin xyz="0 0 0" rpy="0 0 0"/>
-                <geometry>
-                    <sphere radius="${caster_radius}" />
-                </geometry>
-                <material name="black" />
-            </visual>
-        </link>
-    </xacro:macro>
-    <!-- 底盘宏定义 -->
-    <xacro:macro name="mbot_base">
-        <link name="base_footprint">
-            <visual>
-                <origin xyz="0 0 0" rpy="0 0 0" />
-                <geometry>
-                    <box size="0.001 0.001 0.001" />
-                </geometry>
-            </visual>
-        </link>
-        <joint name="base_footprint_joint" type="fixed">
-            <origin xyz="0 0 ${base_length/2 + caster_radius*2}" rpy="0 0 0" />
-            <parent link="base_footprint"/>
-            <child link="base_link" />
-        </joint>
-        <link name="base_link">
-            <visual>
-                <origin xyz=" 0 0 0" rpy="0 0 0" />
-                <geometry>
-                    <cylinder length="${base_length}" radius="${base_radius}"/>
-                </geometry>
-                <material name="yellow" />
-            </visual>
-        </link>
-        <!-- 调用轮子宏 -->
-        <xacro:wheel prefix="left" reflect="-1"/>
-        <xacro:wheel prefix="right" reflect="1"/>
-        <!-- 调用脚轮宏 -->
-        <xacro:caster prefix="front" reflect="-1"/>
-        <xacro:caster prefix="back" reflect="1"/>
-    </xacro:macro>
+<robot name="mbot_base" xmlns:xacro="http://www.ros.org/wiki/xacro">
+    <xacro:include filename="$(find simulation_learning)/models/xacro/base.xacro" />
     <!-- 调用底盘宏 -->
-    <xacro:mbot_base/>
+    <xacro:mbot_base />
 </robot>

File: src/simulation_learning/models/xacro/mbot_with_camera.xacro (robot description, xacro)
@@ -1,16 +1,18 @@
 <?xml version="1.0"?>
-<robot name="arm" xmlns:xacro="http://www.ros.org/wiki/xacro">
-    <xacro:include filename="$(find simulation_learning)/models/xacro/mbot_base.xacro" />
+<robot name="mbot_with_camera" xmlns:xacro="http://www.ros.org/wiki/xacro">
+    <xacro:include filename="$(find simulation_learning)/models/xacro/base.xacro" />
     <xacro:include filename="$(find simulation_learning)/models/xacro/sensors/camera.xacro" />
-    <xacro:property name="camera_offset_x" value="0.17" />
+    <xacro:property name="camera_offset_x" value="0.18" />
     <xacro:property name="camera_offset_y" value="0" />
-    <xacro:property name="camera_offset_z" value="0.10" />
-    <mbot_base/>
+    <xacro:property name="camera_offset_z" value="0.055" />
+    <!-- 调用base宏 -->
+    <xacro:mbot_base />
     <!-- Camera -->
     <joint name="camera_joint" type="fixed">
         <origin xyz="${camera_offset_x} ${camera_offset_y} ${camera_offset_z}" rpy="0 0 0" />
-        <parent link="base_link"/>
-        <child link="camera_link"/>
+        <parent link="base_link" />
+        <child link="camera_link" />
     </joint>
-    <xacro:usb_camera prefix="camera"/>
+    <!-- 调用Camera宏 -->
+    <xacro:usb_camera prefix="camera" />
 </robot>

File: src/simulation_learning/models/xacro/sensors/camera.xacro (robot description, xacro)
@@ -1,12 +1,14 @@
 <?xml version="1.0"?>
-<robot xmlns:xacro="http://www.ros.org/wiki/xacro" name="camera">
+<robot name="camera" xmlns:xacro="http://www.ros.org/wiki/xacro">
     <xacro:macro name="usb_camera" params="prefix:=camera">
         <link name="${prefix}_link">
             <visual>
-                <origin xyz=" 0 0 0 " rpy="0 0 0" />
+                <origin xyz=" 0 0 0 " rpy="0 1.57 0" />
                 <geometry>
-                    <box size="0.01 0.04 0.04" />
+                    <cylinder radius="0.02" length="0.05" />
                 </geometry>
-                <material name="black"/>
+                <material name="gray">
+                    <color rgba="0.25 0.25 0.25 0.95" />
+                </material>
             </visual>
         </link>
