Commit message: code of xacro improve urdf

File: src/simulation_learning/models/xacro/base.xacro (robot description, xacro)
@@ -9,5 +9,4 @@
     <xacro:property name="wheel_joint_y" value="0.19" />
     <xacro:property name="wheel_joint_z" value="0.05" />
-    <!-- wheel_radius - ( base_length/2 - wheel_joint_z) -->
     <xacro:property name="caster_radius" value="0.015" />
     <xacro:property name="caster_joint_x" value="0.18" />
@@ -20,5 +19,8 @@
     </material>
     <material name="gray">
-        <color rgba="0.75 0.75 0.75 1" />
+        <color rgba="0.25 0.25 0.25 0.95" />
+    </material>
+    <material name="white">
+        <color rgba="1 1 1 0.9" />
     </material>
     <!-- 轮子宏定义 -->
@@ -36,5 +38,5 @@
                     <cylinder radius="${wheel_radius}" length="${wheel_length}" />
                 </geometry>
-                <material name="gray" />
+                <material name="white" />
             </visual>
         </link>
@@ -76,5 +78,5 @@
         <link name="base_link">
             <visual>
-                <origin xyz=" 0 0 0" rpy="0 0 0" />
+                <origin xyz="0 0 0" rpy="0 0 0" />
                 <geometry>
                     <cylinder length="${base_length}" radius="${base_radius}" />

File: src/simulation_learning/models/xacro/sensors/laser.xacro (robot description, xacro)
@@ -1,10 +1,10 @@
 <?xml version="1.0"?>
-<robot name="camera" xmlns:xacro="http://www.ros.org/wiki/xacro">
-    <xacro:macro name="usb_camera" params="prefix:=camera">
+<robot name="laser" xmlns:xacro="http://www.ros.org/wiki/xacro">
+    <xacro:macro name="laser" params="prefix:=laser">
         <link name="${prefix}_link">
             <visual>
-                <origin xyz="0 0 0 " rpy="0 1.57 0" />
+                <origin xyz="0 0 0 " rpy="0 0 0" />
                 <geometry>
-                    <cylinder radius="0.02" length="0.05" />
+                    <cylinder length="0.05" radius="0.05" />
                 </geometry>
                 <material name="gray">

File: src/simulation_learning/models/xacro/sensors/laser_gazebo.xacro (robot description, xacro)
@@ -1,5 +1,5 @@
 <?xml version="1.0"?>
 <robot xmlns:xacro="http://www.ros.org/wiki/xacro" name="laser">
-    <xacro:macro name="rplidar" params="prefix:=laser">
+    <xacro:macro name="laser" params="prefix:=laser">
         <!-- Create laser reference frame -->
         <link name="${prefix}_link">
@@ -29,5 +29,5 @@
         </gazebo>
         <gazebo reference="${prefix}_link">
-            <sensor type="ray" name="rplidar">
+            <sensor type="ray" name="laser">
                 <pose>0 0 0 0 0 0</pose>
                 <visualize>false</visualize>
@@ -53,5 +53,5 @@
                     </noise>
                 </ray>
-                <plugin name="gazebo_rplidar" filename="libgazebo_ros_laser.so">
+                <plugin name="gazebo_laser" filename="libgazebo_ros_laser.so">
                     <topicName>/scan</topicName>
                     <frameName>laser_link</frameName>

Commit message: xacro模型 移到地面以上

File: src/simulation_learning/models/xacro/base.xacro (robot description, xacro)
@@ -8,5 +8,4 @@
     <xacro:property name="wheel_length" value="0.025" />
     <xacro:property name="wheel_joint_y" value="0.19" />
-    <xacro:property name="wheel_joint_z" value="0.05" />
     <xacro:property name="caster_radius" value="0.015" />
     <xacro:property name="caster_joint_x" value="0.18" />
@@ -27,5 +26,5 @@
     <xacro:macro name="wheel" params="prefix reflect">
         <joint name="${prefix}_wheel_joint" type="continuous">
-            <origin xyz="0 ${reflect*wheel_joint_y} ${-wheel_joint_z}" rpy="0 0 0" />
+            <origin xyz="0 ${reflect*wheel_joint_y} ${wheel_radius}" rpy="0 0 0" />
             <parent link="base_link" />
             <child link="${prefix}_wheel_link" />
@@ -45,5 +44,5 @@
     <xacro:macro name="caster" params="prefix reflect">
         <joint name="${prefix}_caster_joint" type="continuous">
-            <origin xyz="${reflect*caster_joint_x} 0 ${-(base_length/2 + caster_radius)}"
+            <origin xyz="${reflect*caster_joint_x} 0 ${caster_radius}"
                 rpy="0 0 0" />
             <parent link="base_link" />
@@ -63,20 +62,7 @@
     <!-- 底盘宏定义 -->
     <xacro:macro name="mbot_base">
-        <link name="base_footprint">
-            <visual>
-                <origin xyz="0 0 0" rpy="0 0 0" />
-                <geometry>
-                    <box size="0.001 0.001 0.001" />
-                </geometry>
-            </visual>
-        </link>
-        <joint name="base_footprint_joint" type="fixed">
-            <origin xyz="0 0 ${base_length/2 + caster_radius*2}" rpy="0 0 0" />
-            <parent link="base_footprint" />
-            <child link="base_link" />
-        </joint>
         <link name="base_link">
             <visual>
-                <origin xyz="0 0 0" rpy="0 0 0" />
+                <origin xyz="0 0 ${2*caster_radius + base_length/2}" rpy="0 0 0" />
                 <geometry>
                     <cylinder length="${base_length}" radius="${base_radius}" />

File: src/simulation_learning/models/xacro/mbot_with_laser_camera.xacro (robot description, xacro)
@@ -6,8 +6,8 @@
     <xacro:property name="laser_offset_x" value="0" />
     <xacro:property name="laser_offset_y" value="0" />
-    <xacro:property name="laser_offset_z" value="0.105" />
+    <xacro:property name="laser_offset_z" value="${2*caster_radius + base_length + laser_length/2}" />
     <xacro:property name="camera_offset_x" value="0.18" />
     <xacro:property name="camera_offset_y" value="0" />
-    <xacro:property name="camera_offset_z" value="0.055" />
+    <xacro:property name="camera_offset_z" value="0.165" />
     <!-- 调用base宏 -->
     <xacro:mbot_base />

File: src/simulation_learning/models/xacro/sensors/laser.xacro (robot description, xacro)
@@ -1,4 +1,6 @@
 <?xml version="1.0"?>
 <robot name="laser" xmlns:xacro="http://www.ros.org/wiki/xacro">
+    <xacro:property name="laser_radius" value="0.05" />
+    <xacro:property name="laser_length" value="0.05" />
     <xacro:macro name="laser" params="prefix:=laser">
         <link name="${prefix}_link">
@@ -6,5 +8,5 @@
                 <origin xyz="0 0 0 " rpy="0 0 0" />
                 <geometry>
-                    <cylinder length="0.05" radius="0.05" />
+                    <cylinder length="${laser_length}" radius="${laser_radius}" />
                 </geometry>
                 <material name="gray">
