Commit message: 更新rviz配置

File: src/simulation_learning/models/xacro/mbot_with_camera.xacro (robot description, xacro)
@@ -5,5 +5,5 @@
     <xacro:property name="camera_offset_x" value="0.18" />
     <xacro:property name="camera_offset_y" value="0" />
-    <xacro:property name="camera_offset_z" value="0.055" />
+    <xacro:property name="camera_offset_z" value="0.165" />
     <!-- 调用base宏 -->
     <xacro:mbot_base />
